File: staor_v2/staor_v2.kicad_pcb (KiCad board)
At the start: 4 copper layers, 109.2 x 118.1 mm, 3 parts

Commit message: cut layer
Parts:
- added REF**: MountingHole_2.1mm, MountingHole:MountingHole_2.1mm, F.Cu at (140.0, 115.5)
- added REF**: MountingHole_2.1mm, MountingHole:MountingHole_2.1mm, F.Cu at (162.0, 110.0)
- added REF**: MountingHole_2.1mm, MountingHole:MountingHole_2.1mm, F.Cu at (156.0, 83.0)
- added REF**: MountingHole_2.1mm, MountingHole:MountingHole_2.1mm, F.Cu at (132.5, 91.5)
Other:
- board size 109.2 x 118.1 mm -> 119 x 119 mm
